File: Wiring_Heatpump/Wiring.sch (EAGLE design)
At the start: 16 parts, among them P1 Lichtstrom, P2 Heizstrom

Commit message: manuell schaltbare EVU-Abschaltung hinzugefügt
Parts:
- added JP1, JP2, JP3, JP4, JP5, JP6: (no value), pinhead:PINHD-1X1
- added K4, K6, K8: (no value), e-schuetze-relais:HILFSSCHUETZ_11-12
- added K5, K7, K9: (no value), e-schuetze-relais:HILFSSCHUETZ_13-14
- added R1, R2, R7: (no value), ptc-ntc:NTC644A
- added R3, R4, R8: (no value), rcl:R-EU_0204/2V
- added R5, R6, R9: 330R, rcl:R-EU_0204/2V
Connections:
- new net N$29: K41.1, K51.4, R1.1, R5.1
- new net N$30: JP2.1, K41.2, R5.2
- new net N$31: JP1.1, R1.2, R4.1
- new net N$32: K51.3, R4.2
- new net N$33: K61.1, K71.4, R2.1, R6.1
- new net N$34: K61.2, R6.2
- new net N$35: R2.2, R3.1
- new net N$36: K71.3, R3.2
- new net N$37: K81.1, K91.4, R7.1, R9.1
- new net N$38: K81.2, R9.2
- new net N$39: R7.2, R8.1
- new net N$40: K91.3, R8.2
Other:
- note added: "Heizstromumschaltung"
- note added: "TB (Warmwasser)"
- note added: "TPM (Heizung mitte)"
- note added: "TPO (Heizung oben)"
- note added: "Warmwassertemperatur"
